File: schematics/omi/omi.kicad_sch (KiCad schematic)
At the start: 36 parts, among them J1 AudioJack4, J2 AudioJack4, U1 ESP32-S3-WROOM-1, U2 XIAO-nRF52840-SMD, X1 PCM510XA

Commit message: feat: Update schematics for common xtal
Connections:
- net AUDIO_LRCK is gone; now on net COM_XTAL: U1.5 (IO5), X1.15 (LRCK)
- net COM_XTAL: now reaches U2.1 (P0.02_A0_D0)
Other:
- note added: "open-helmet"
- note removed: "omi"
Changed lines of the file:
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@@
 		(rev "0.1")
 	)
-	(text "omi"
+	(text "open-helmet"
 		(exclude_from_sim no)
 		(at 229.108 172.72 0)
@@
 	(wire
 		(pts
+			(xy 146.05 87.63) (xy 156.21 87.63)
+		)
+		(stroke
+			(width 0)
+			(type default)
+		)
+	)
+	(wire
+		(pts
 			(xy 139.7 39.37) (xy 149.86 39.37)
 		)
@@
 		)
 	)
-	(label "AUDIO_LRCK"
+	(label "COM_XTAL"
 		(at 40.64 57.15 0)
 		(effects
@@
 		)
 	)
-	(label "AUDIO_LRCK"
+	(label "COM_XTAL"
 		(at 224.79 109.22 0)
 		(effects
@@
 		(effects
 			(font
+				(size 1.27 1.27)
+			)
+			(justify left bottom)
+		)
+	)
+	(label "COM_XTAL"
+		(at 146.05 87.63 0)
+		(effects
+			(font
