File: schematics/omi/omi.kicad_sch (KiCad schematic)
At the start: 36 parts, among them J1 AudioJack4, J2 AudioJack4, U1 ESP32-S3-WROOM-1, U2 XIAO-nRF52840-SMD, X1 PCM510XA

Commit message: feat: publish final OMI v1 hardware
Parts:
- removed C1: 0.47uF, Adafruit MAX9814:C0805K, symbol Adafruit MAX9814-eagle-import:C-USC0805K
- removed C13, C15, C19, C22: 10uF, Adafruit PCM510x I2S DAC:0805-NO, symbol Adafruit PCM510x I2S DAC-eagle-import:CAP_CERAMIC0805-NOOUTLINE
- removed C14, C16, C20, C21: 0.1uF, Adafruit PCM510x I2S DAC:0603-NO, symbol Adafruit PCM510x I2S DAC-eagle-import:CAP_CERAMIC0603_NO
- removed C17, C18: 2.2uF, Adafruit PCM510x I2S DAC:0603-NO, symbol Adafruit PCM510x I2S DAC-eagle-import:CAP_CERAMIC0603_NO
- removed C2, C9: 0.1uF, Adafruit MAX9814:C0805K, symbol Adafruit MAX9814-eagle-import:C-USC0805K
- removed C3, C5: 2.2uF, Adafruit MAX9814:C0805K, symbol Adafruit MAX9814-eagle-import:C-USC0805K
- removed C7, C8: 2.2nF, Adafruit PCM510x I2S DAC:0603-NO, symbol Adafruit PCM510x I2S DAC-eagle-import:CAP_CERAMIC0603_NO
- removed FB1: Ferrite, Adafruit PCM510x I2S DAC:0603-NO, symbol Adafruit PCM510x I2S DAC-eagle-import:FERRITE-0603NO
- removed FB2: FERRITE, Adafruit MAX9814:0805, symbol Adafruit MAX9814-eagle-import:FERRITE0805
- removed J1, J2: AudioJack4, symbol Connector_Audio:AudioJack4
- removed NT1: NetTie_2, symbol Device:NetTie_2
- removed R1, R10, R2, R8, R9: 10k, Adafruit PCM510x I2S DAC:0603-NO, symbol Adafruit PCM510x I2S DAC-eagle-import:RESISTOR_0603_NOOUT
- removed R11: 150k, Adafruit MAX9814:R0805, symbol Adafruit MAX9814-eagle-import:R-US_R0805
- removed R3: 2.2K, Adafruit MAX9814:R0805, symbol Adafruit MAX9814-eagle-import:R-US_R0805
- removed R4, R6: 470, Adafruit PCM510x I2S DAC:0603-NO, symbol Adafruit PCM510x I2S DAC-eagle-import:RESISTOR_0603_NOOUT
- removed R5: 100k, Adafruit MAX9814:R0805, symbol Adafruit MAX9814-eagle-import:R-US_R0805
- removed U$1: MAX9814TDFN14, Adafruit MAX9814:TDFN14_3X3MM, symbol Adafruit MAX9814-eagle-import:MAX9814TDFN14
- removed U2: XIAO-nRF52840-SMD, Seeed_Studio_XIAO_Series:XIAO-nRF52840-SMD, symbol Seeed_Studio_XIAO_Series:XIAO-nRF52840-SMD
- removed X1: PCM510XA, Adafruit PCM510x I2S DAC:TSSOP20, symbol Adafruit PCM510x I2S DAC-eagle-import:PCM510XA
- U1: LCSC (none) -> C2913198; MNF PART NUMBER (none) -> ESP32-S3-WROOM-1-N8; Manufacturer (none) -> Espressif Systems
Connections:
- net COM_XTAL: now also U1.28 (IO35)
- net ESP_USB_D-: now reaches U1.13 (USB_D-)
- net ESP_USB_D+: now reaches U1.14 (USB_D+)
- net NRF_MOSI: now reaches U1.21 (IO13)
- net NRF_SWDIO: now reaches U1.22 (IO14)
- net USB_HIGH_CURRENT: now reaches U1.23 (IO21)
- net ESP_BOOT: now reaches U1.27 (IO0)
- net ESP_EN: now reaches U1.3 (EN)
- net ESP_UART_RX: now reaches U1.36 (RXD0)
- net ESP_UART_TX: now reaches U1.37 (TXD0)
- net NRF_SWDCLK: now reaches U1.8 (IO15)
- net NRF_RESET: now reaches U1.9 (IO16)
- no-connect marks 2 -> 17
Other:
- added sheet Audio (Audio.kicad_sch)
- added sheet Radio (Radio.kicad_sch)
- added sheet USB_Power (USB_Power.kicad_sch)
- moved on the sheet: U1
