File: schematics/omi/Radio.kicad_sch (KiCad schematic)
At the start: 37 parts, among them J3 NRF SWD RECOVERY, U2 NRF52840-QIAA-R, U3 NRF21540-QDAA-R, Y1 32MHz 8pF, Y2 32.768kHz 12.5pF

Commit message: fix: synchronize KiCad design and repair 3D models
Parts:
- J3: now left out of the parts list
Changed lines of the file:
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@@
 		(body_style 1)
 		(exclude_from_sim no)
-		(in_bom yes)
+		(in_bom no)
 		(on_board yes)
-		(in_pos_files yes)
+		(in_pos_files no)
 		(dnp no)
 		(property "Reference" "J3"
