File: schematics/omi/omi.kicad_pcb (KiCad board)
At the start: 4 copper layers, 100 x 50 mm, 117 parts, among them J3 NRF SWD RECOVERY, J4 TYPE-C-31-M-12, J5 LiPo + NTC, J6 PJ-327C-4A Headphones, J7 PJ-327C-4A Microphone, J8 ESP FACTORY, SW1 ESP RESET, SW2 ESP BOOT, SW3 POWER ON/OFF, U1 ESP32-S3-WROOM-1, U2 NRF52840-QIAA-R, U3 NRF21540-QDAA-R, U4 BQ24074RGTR, U5 TPS63020DSJR, U6 USBLC6-2SC6, U7 PCM5102APWR, U8 MAX9814ETD+T, U9 TPA6132A2RTER, Y1 32MHz 8pF, Y2 32.768kHz 12.5pF

Commit message: fix: synchronize KiCad design and repair 3D models
Parts:
- J4: value TYPE-C-31-M-12 -> USB-C
Connections:
- net ANT_TUNED renamed /Radio/ANT_TUNED
- net AUDIO_BCK renamed /AUDIO_BCK
- net AUDIO_DIN renamed /AUDIO_DIN
- net BAT+ renamed /USB_Power/BAT+
- net BAT_NTC renamed /USB_Power/BAT_NTC
- net CHG_ISET renamed /USB_Power/CHG_ISET
- net CHG_ITERM renamed /USB_Power/CHG_ITERM
- net CHG_TMR renamed /USB_Power/CHG_TMR
- net COM_XTAL renamed /COM_XTAL
- net ESP_BOOT renamed /ESP_BOOT
- net ESP_EN renamed /ESP_EN
- net ESP_UART_RX renamed /ESP_UART_RX
- net ESP_UART_TX renamed /ESP_UART_TX
- net ESP_USB_D+ renamed /ESP_USB_D+
- net ESP_USB_D- renamed /ESP_USB_D-
- net FEM_ANT1_MID renamed /Radio/FEM_ANT1_MID
- net FEM_ANT1_RAW renamed /Radio/FEM_ANT1_RAW
- net FEM_ANT2_RAW renamed /Radio/FEM_ANT2_RAW
- net FEM_ANT_SEL renamed /Radio/FEM_ANT_SEL
- net FEM_CSN renamed /Radio/FEM_CSN
- net FEM_MISO renamed /Radio/FEM_MISO
- net FEM_MODE renamed /Radio/FEM_MODE
- net FEM_MODE_RAW renamed /Radio/FEM_MODE_RAW
- net FEM_MOSI renamed /Radio/FEM_MOSI
- net FEM_PDN renamed /Radio/FEM_PDN
- net FEM_RF_50R renamed /Radio/FEM_RF_50R
- net FEM_RX_EN renamed /Radio/FEM_RX_EN
- net FEM_SCK renamed /Radio/FEM_SCK
- net FEM_TRX renamed /Radio/FEM_TRX
- net FEM_TX_EN renamed /Radio/FEM_TX_EN
- net HP_CP_N renamed /Audio/HP_CP_N
- net HP_CP_P renamed /Audio/HP_CP_P
- net HP_EN renamed /Audio/HP_EN
- net HP_GND renamed /Audio/HP_GND
- net HP_L_IN renamed /Audio/HP_L_IN
- net HP_OUT_L renamed /Audio/HP_OUT_L
- net HP_OUT_R renamed /Audio/HP_OUT_R
- net HP_R_IN renamed /Audio/HP_R_IN
- net HP_VDD renamed /Audio/HP_VDD
- net HP_VSS renamed /Audio/HP_VSS
- net MIC_BIAS renamed /Audio/MIC_BIAS
- net MIC_BIAS_OUT renamed /Audio/MIC_BIAS_OUT
- net MIC_CG renamed /Audio/MIC_CG
- net MIC_CT renamed /Audio/MIC_CT
- net MIC_IN renamed /Audio/MIC_IN
- net MIC_JACK renamed /Audio/MIC_JACK
- net MIC_OUT renamed /MIC_OUT
- net MIC_PRE_OUT renamed /Audio/MIC_PRE_OUT
- net MIC_TH renamed /Audio/MIC_TH
- net NRF_DCC renamed /Radio/NRF_DCC
- net NRF_DEC1 renamed /Radio/NRF_DEC1
- net NRF_DEC2 renamed /Radio/NRF_DEC2
- net NRF_DEC3 renamed /Radio/NRF_DEC3
- net NRF_DEC4 renamed /Radio/NRF_DEC4
- net NRF_DEC5 renamed /Radio/NRF_DEC5
- net NRF_DEC6 renamed /Radio/NRF_DEC6
- net NRF_DECUSB renamed /Radio/NRF_DECUSB
- net NRF_MISO renamed /NRF_MISO
- net NRF_MOSI renamed /NRF_MOSI
- net NRF_RESET renamed /NRF_RESET
- net NRF_RF_RAW renamed /Radio/NRF_RF_RAW
- net NRF_RX renamed /NRF_RX
- net NRF_SCK renamed /NRF_SCK
- net NRF_SWDCLK renamed /NRF_SWDCLK
- net NRF_SWDCLK_RAW renamed /Radio/NRF_SWDCLK_RAW
- net NRF_SWDIO renamed /NRF_SWDIO
- net NRF_SWDIO_RAW renamed /Radio/NRF_SWDIO_RAW
- net NRF_TX renamed /NRF_TX
- net NRF_XC1 renamed /Radio/NRF_XC1
- net NRF_XC2 renamed /Radio/NRF_XC2
- net NRF_XL1 renamed /Radio/NRF_XL1
- net NRF_XL2 renamed /Radio/NRF_XL2
- net PCM_CP_N renamed /Audio/PCM_CP_N
- net PCM_CP_P renamed /Audio/PCM_CP_P
- net PCM_LDOO renamed /Audio/PCM_LDOO
- net PCM_L_AC renamed /Audio/PCM_L_AC
- net PCM_L_FILT renamed /Audio/PCM_L_FILT
- net PCM_L_RAW renamed /Audio/PCM_L_RAW
- net PCM_R_AC renamed /Audio/PCM_R_AC
- net PCM_R_FILT renamed /Audio/PCM_R_FILT
- net PCM_R_RAW renamed /Audio/PCM_R_RAW
- net PCM_VNEG renamed /Audio/PCM_VNEG
- net PWR_ENABLE renamed /USB_Power/PWR_ENABLE
- net REG_FB renamed /USB_Power/REG_FB
- net REG_L1 renamed /USB_Power/REG_L1
- net REG_L2 renamed /USB_Power/REG_L2
- net REG_PG renamed /USB_Power/REG_PG
- net SYS_OUT renamed /USB_Power/SYS_OUT
- net USB_CC1 renamed /USB_Power/USB_CC1
- net USB_CC2 renamed /USB_Power/USB_CC2
- net USB_D+_CONN renamed /USB_Power/USB_D+_CONN
- net USB_D+_PROTECTED renamed /USB_Power/USB_D+_PROTECTED
- net USB_D-_CONN renamed /USB_Power/USB_D-_CONN
- net USB_D-_PROTECTED renamed /USB_Power/USB_D-_PROTECTED
- net USB_HIGH_CURRENT renamed /USB_HIGH_CURRENT
- net USB_SHIELD renamed /USB_Power/USB_SHIELD
- net VBUS renamed /USB_Power/VBUS
- U1 pad 10: (no net) -> unconnected-(U1-IO17-Pad10)
- U1 pad 11: (no net) -> unconnected-(U1-IO18-Pad11)
- U1 pad 12: (no net) -> unconnected-(U1-IO8-Pad12)
- U1 pad 15: (no net) -> unconnected-(U1-IO3-Pad15)
- U1 pad 16: (no net) -> unconnected-(U1-IO46-Pad16)
- U1 pad 24: (no net) -> unconnected-(U1-IO47-Pad24)
- U1 pad 25: (no net) -> unconnected-(U1-IO48-Pad25)
- U1 pad 26: (no net) -> unconnected-(U1-IO45-Pad26)
- U1 pad 29: (no net) -> unconnected-(U1-IO36-Pad29)
- U1 pad 30: (no net) -> unconnected-(U1-IO37-Pad30)
- U1 pad 31: (no net) -> unconnected-(U1-IO38-Pad31)
- U1 pad 32: (no net) -> unconnected-(U1-IO39-Pad32)
- U1 pad 33: (no net) -> unconnected-(U1-IO40-Pad33)
- U1 pad 34: (no net) -> unconnected-(U1-IO41-Pad34)
- U1 pad 35: (no net) -> unconnected-(U1-IO42-Pad35)
- U1 pad 38: (no net) -> unconnected-(U1-IO2-Pad38)
- U1 pad 6: (no net) -> unconnected-(U1-IO6-Pad6)
